File: PCB/PSOC_5_PCB/Main Microcontroller.kicad_sch (KiCad schematic)
At the start: 60 parts, among them IC1 CY8C5888LTI-LP097, J1 USB_B_Micro, J10 GPIO Pins 7, J11 GPIO Pins 6, J12 GPIO Pins 2, J13 GPIO Pins 3, J14 GPIO Pins 5, J16 GPIO Pins 4, J2 Program Upload Interface, J3 Debug Print Interface, J4 RPI UART, J5 OEM UART, J6 Pressure Before ΔΣ, J7 SAR ADC, J8 Pressure After ΔΣ, J9 GPIO Pins 1, SW1 RESET_BUTTON

Commit message: PCB Layout Pushed
Parts:
- removed J10: GPIO Pins 7, Connector_PinHeader_2.54mm:PinHeader_1x06_P2.54mm_Vertical, symbol Connector:Conn_01x06_Pin
- removed J11: GPIO Pins 6, Connector_PinHeader_2.54mm:PinHeader_2x04_P2.54mm_Vertical, symbol Connector_Generic:Conn_02x04_Top_Bottom
- removed J12: GPIO Pins 2, Connector_PinHeader_2.54mm:PinHeader_1x04_P2.54mm_Vertical, symbol Connector:Conn_01x04_Pin
- removed J13: GPIO Pins 3, Connector_PinHeader_2.54mm:PinHeader_1x04_P2.54mm_Vertical, symbol Connector:Conn_01x04_Pin
- removed J14: GPIO Pins 5, Connector_PinHeader_2.54mm:PinHeader_1x05_P2.54mm_Vertical, symbol Connector:Conn_01x05_Pin
- removed J16: GPIO Pins 4, Connector_PinHeader_2.54mm:PinHeader_1x06_P2.54mm_Vertical, symbol Connector:Conn_01x06_Pin
- removed J2: Program Upload Interface, Connector_PinHeader_2.54mm:PinHeader_1x05_P2.54mm_Vertical, symbol Connector:Conn_01x05_Pin
- removed J3: Debug Print Interface, Connector_PinHeader_2.54mm:PinHeader_1x02_P2.54mm_Vertical, symbol Connector:Conn_01x02_Pin
- removed J4: RPI UART, Connector_PinHeader_2.54mm:PinHeader_1x03_P2.54mm_Vertical, symbol Connector:Conn_01x03_Pin
- removed J5: OEM UART, Connector_PinHeader_2.54mm:PinHeader_1x03_P2.54mm_Vertical, symbol Connector:Conn_01x03_Pin
- removed J6: Pressure Before ΔΣ, Connector_PinHeader_2.54mm:PinHeader_1x03_P2.54mm_Vertical, symbol Connector:Conn_01x03_Pin
- removed J7: SAR ADC, Connector_PinSocket_2.54mm:PinSocket_1x05_P2.54mm_Vertical, symbol Connector:Conn_01x05_Pin
- removed J8: Pressure After ΔΣ, Connector_PinHeader_2.54mm:PinHeader_1x03_P2.54mm_Vertical, symbol Connector:Conn_01x03_Pin
- removed J9: GPIO Pins 1, Connector_PinHeader_2.54mm:PinHeader_1x05_P2.54mm_Vertical, symbol Connector:Conn_01x05_Pin
- removed R18, R19: 10KΩ, Resistor_SMD:R_0402_1005Metric, symbol Device:R
- removed R8: 0Ω, Resistor_SMD:R_0402_1005Metric, symbol Device:R
- added C22, C23, C24, C25, C26, C28, C29: 10uF, Capacitor_SMD:C_0805_2012Metric, symbol Device:C
- added C30, C31, C32: 1uF, Capacitor_SMD:C_0603_1608Metric, symbol Device:C
- added D3: D_Schottky_KKA, Package_TO_SOT_SMD:SOT-23, symbol Device:D_Schottky_KKA
- added J10: GPIO_2, Connector_JST:JST_GH_BM09B-GHS-TBT_1x09-1MP_P1.25mm_Vertical, symbol Connector_Generic:Conn_01x09
- added J11: GPIO_3, Connector_JST:JST_GH_BM07B-GHS-TBT_1x07-1MP_P1.25mm_Vertical, symbol Connector_Generic:Conn_01x07
- added J12: GPIO_4, Connector_JST:JST_GH_BM05B-GHS-TBT_1x05-1MP_P1.25mm_Vertical, symbol Connector_Generic:Conn_01x05
- added J13: GPIO_5, Connector_JST:JST_GH_BM05B-GHS-TBT_1x05-1MP_P1.25mm_Vertical, symbol Connector_Generic:Conn_01x05
- added J14: I2C_1, Connector_JST:JST_GH_BM04B-GHS-TBT_1x04-1MP_P1.25mm_Vertical, symbol Connector_Generic:Conn_01x04
- added J15: Power Jumper, Connector_PinHeader_2.54mm:PinHeader_1x03_P2.54mm_Vertical, symbol Connector:Conn_01x03_Pin
- added J2: Program_Upload_Interface, Connector_JST:JST_GH_BM05B-GHS-TBT_1x05-1MP_P1.25mm_Vertical, symbol Connector_Generic:Conn_01x05
- added J3: Debug_Interface, Connector_JST:JST_GH_BM02B-GHS-TBT_1x02-1MP_P1.25mm_Vertical, symbol Connector_Generic:Conn_01x02
- added J4: SAR_ADC, Connector_JST:JST_GH_BM06B-GHS-TBT_1x06-1MP_P1.25mm_Vertical, symbol Connector_Generic:Conn_01x06
- added J5: ΔΣ Pressure Before Gas Exchange, Connector_JST:JST_GH_BM04B-GHS-TBT_1x04-1MP_P1.25mm_Vertical, symbol Connector_Generic:Conn_01x04
- added J6: ΔΣ Pressure After Gas Exchange, Connector_JST:JST_GH_BM04B-GHS-TBT_1x04-1MP_P1.25mm_Vertical, symbol Connector_Generic:Conn_01x04
- added J7: OEM_UART, Connector_JST:JST_GH_BM04B-GHS-TBT_1x04-1MP_P1.25mm_Vertical, symbol Connector_Generic:Conn_01x04
- added J8: RPI UART, Connector_JST:JST_GH_BM03B-GHS-TBT_1x03-1MP_P1.25mm_Vertical, symbol Connector_Generic:Conn_01x03
- added J9: GPIO_1, Connector_JST:JST_GH_BM05B-GHS-TBT_1x05-1MP_P1.25mm_Vertical, symbol Connector_Generic:Conn_01x05
- added R13, R24: 4.7KΩ, Resistor_SMD:R_0603_1608Metric, symbol Device:R
- D2: value SOD123 -> PMEG2010ER; footprint Diode_SMD:D_SOD-123 -> Diode_SMD:Nexperia_CFP3_SOD-123W
- F1: footprint (none) -> ECMO:RESC3216X125N
- R1, R10, R11, R3, R4: footprint Resistor_SMD:R_0402_1005Metric -> Resistor_SMD:R_0603_1608Metric
- R12: value 0Ω -> 0Ω(DNI)
- R14: value 10KΩ -> 5KΩ
- R15: value 20KΩ -> 10KΩ
- R22, R23: value 10KΩ -> 2.2KΩ
- R6: footprint Resistor_SMD:R_0402_1005Metric -> Resistor_SMD:R_0805_2012Metric
- R7: value 0Ω -> 1KΩ
- U1: renamed from IC1; footprint CY8C5888LTI-LP097:QFN40P800X800X100-69N -> ECMO:QFN-68; DESCRIPTION ARM Microcontrollers - MCU 256KB Flash 64KBSRAM PSoC 5LP -> (none)
Connections:
- net P12.2 is gone; now on net USER_LED: U1.46 (P12[2]_(SIO))
- net P12.3 is gone; now on net TX_Debug: U1.47 (P12[3]_(SIO)
- net P15.0 is gone; now on net RX_RPI: U1.27 ((MHZ_XTAL:_XO,_GPIO)_P15[0])
- net P15.1 is gone; now on net TX_RPI: U1.28 ((MHZ_XTAL:_XI,_GPIO)_P15[1])
- net P2.2 is gone; now on net ADC_CH1: U1.64 (P2[2]_(GPIO))
- net P2.3 is gone; now on net ADC_CH2: U1.65 (P2[3]_(GPIO,_TRACECLK))
- net P2.4 is gone; now on net ADC_CH3: U1.66 (P2[4]_(GPIO,_TRACEDATA[0]))
- net P2.6 is gone; now on net Pressure_Before_Neg: U1.1 ((TRACEDATA[2],_GPIO)_P2[6])
- net P2.7 is gone; now on net Pressure_Before_Pos: U1.2 ((TRACEDATA[3],_GPIO)_P2[7])
- net VDDIO is gone; now on net VDD: C18.1, C19.1, C20.1, C21.1, U1.17 (VDDIO1), U1.35 (VDDIO3), U1.52 (VDDIO0), U1.67 (VDDIO2)
- net ADC_CH0: now also R16.1, U1.63 (P2[1]_(GPIO)), D3.1 (K); no longer R16.2, R20.2, U1.41 (P15[3]_(GPIO,_KHZ_XTAL:_XI))
- net ADC_CH1: now also R17.1, D3.2 (K); no longer R17.2, R21.2, U1.32 ((OPAMP3+,_GPIO)_P3[3])
- net ADC_CH2: now also R21.2; no longer U1.37 (P3[7]_(GPIO,_OPAMP3OUT))
- net ADC_CH3: now also R20.2; no longer U1.56 (P0[7]_(GPIO,_IDAC2))
- net DM: now also R4.1; no longer R4.2
- net DM_P: now also R4.2; no longer R4.1
- net DP: now also R1.1; no longer R1.2
- net DP_P: now also R1.2; no longer R1.1
- net GND: now also R7.2, C22.2, C23.2, C24.2, C25.2, C26.2, C28.2, C29.2, C30.2, C31.2, C32.2, D3.3 (A), J10.1 (Pin_1), J11.1 (Pin_1), J12.1 (Pin_1), J13.1 (Pin_1), J14.4 (Pin_4), J2.4 (Pin_4), J3.2 (Pin_2), J4.5 (Pin_5), J4.6 (Pin_6), J5.4 (Pin_4), J6.4 (Pin_4), J7.1 (Pin_1), J8.3 (Pin_3), J9.1 (Pin_1); no longer R22.1, R23.1, SW1.2
- net P0.0: now also J12.5 (Pin_5)
- net P0.1: now also J12.4 (Pin_4)
- net P0.2: now also J12.3 (Pin_3)
- net P0.3: now also J12.2 (Pin_2)
- net P0.4: now also U1.53 (P0[4]_(GPIO,_OPAMP2+,_SAR0_EXTREF)), J13.5 (Pin_5)
- net P0.6: now also J13.3 (Pin_3)
- net P1.2: now also J9.5 (Pin_5)
- net P1.3: now also J9.4 (Pin_4)
- net P1.4: now also J9.3 (Pin_3)
- net P1.5: now also J9.2 (Pin_2)
- net P15.2: now also J11.3 (Pin_3)
- net P3.0: now also J10.7 (Pin_7)
- net P3.1: now also J10.6 (Pin_6)
- net P3.2: now also J10.5 (Pin_5)
- net P3.6: now also J11.7 (Pin_7)
- net PROG_RESET: now also J2.3 (Pin_3)
- net Pressure_After_Neg: now also U1.60 (P15[4]_(GPIO)), J6.3 (Pin_3); no longer U1.54 (P0[5]_(GPIO,_OPAMP2-))
- net Pressure_After_Pos: now also U1.61 (P15[5]_(GPOI)), J6.2 (Pin_2); no longer U1.53 (P0[4]_(GPIO,_OPAMP2+,_SAR0_EXTREF))
- net Pressure_Before_Neg: now also J5.3 (Pin_3); no longer U1.33 ((OPAMP1-,_GPIO)_P3[4])
- net Pressure_Before_Pos: now also J5.2 (Pin_2); no longer U1.34 ((OPAMP1+,_GPIO)_P3[5])
- net RX_OEM: now also U1.20 ((SIO)_P12[6]), J7.3 (Pin_3); no longer U1.18 ((GPIO)_P1[6])
- net RX_RPI: now also J8.2 (Pin_2); no longer U1.60 (P15[4]_(GPIO))
- net TX_Debug: no longer U1.21 ((SIO)_P12[7])
- net TX_OEM: now also U1.21 ((SIO)_P12[7]), J7.2 (Pin_2); no longer U1.19 ((GPIO)_P1[7])
- net TX_RPI: no longer U1.61 (P15[5]_(GPOI))
- net USER_LED: no longer U1.63 (P2[1]_(GPIO))
- net VDD: now also R6.2, C22.1, C23.1, C24.1, C25.1, C26.1, C28.1, C29.1, C30.1, C31.1, C32.1, J14.1 (Pin_1), J5.1 (Pin_1), J6.1 (Pin_1), J7.4 (Pin_4), R13.1, R24.2; no longer R7.2
- net VTARG: now also J15.1 (Pin_1), J2.5 (Pin_5); no longer D2.1 (K), R6.1
- net at R12.1, R14.1, R15.1: now also J8.1 (Pin_1)
- net at R7.1: now also SW1.2; no longer R6.2
- net at R9.1: now also J3.1 (Pin_1)
- net Earth GND renamed USB_SHIELD
- net I2C_SCL renamed SCL1
- net SCL1: now also J11.5 (Pin_5)
- net I2C_SDA renamed SDA1
- net SDA1: now also J11.4 (Pin_4)
- net P1.0 renamed PROG_SWDIO
- net PROG_SWDIO: now also J2.1 (Pin_1)
- net P1.1 renamed PROG_SWDCLK
- net PROG_SWDCLK: now also J2.2 (Pin_2)
- net P12.4 renamed SCL2
- net SCL2: now also J14.3 (Pin_3), R13.2
- net P12.5 renamed SDA2
- net SDA2: now also J14.2 (Pin_2), R24.1
- net P2.0: no longer names the net of U1.62 (P2[0]_(GPIO))
- net P2.5: no longer names the net of U1.68 (P2[5]_(GPIO,_TRACEDATA[1]))
- new net: J15.2 (Pin_2), R6.1
- new net: J4.1 (Pin_1), R23.1
- new net: J4.3 (Pin_3), R17.2
- new net: J4.2 (Pin_2), R22.1
- new net: J4.4 (Pin_4), R16.2
- new net P0.5: J13.4 (Pin_4), U1.54 (P0[5]_(GPIO,_OPAMP2-))
- new net P0.7: J13.2 (Pin_2), U1.56 (P0[7]_(GPIO,_IDAC2))
- new net P1.6: J10.9 (Pin_9), U1.18 ((GPIO)_P1[6])
- new net P1.7: J10.8 (Pin_8), U1.19 ((GPIO)_P1[7])
- new net P15.3: J11.2 (Pin_2), U1.41 (P15[3]_(GPIO,_KHZ_XTAL:_XI))
- new net P3.3: J10.4 (Pin_4), U1.32 ((OPAMP3+,_GPIO)_P3[3])
- new net P3.4: J10.3 (Pin_3), U1.33 ((OPAMP1-,_GPIO)_P3[4])
- new net P3.5: J10.2 (Pin_2), U1.34 ((OPAMP1+,_GPIO)_P3[5])
- new net P3.7: J11.6 (Pin_6), U1.37 (P3[7]_(GPIO,_OPAMP3OUT))
- new net VBUS: D2.1 (K), J15.3 (Pin_3)
- no-connect marks 3 -> 4
Other:
- note added: "Additional Decoupling Capacitor"
- note added: "Free Headers"
- note removed: "Extra GPIO"
- moved on the sheet: C10, C11, C12, C13, C14, C15, C16, C17, C18, C3, C4, C7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
Changed lines of the file:
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@@
 (kicad_sch
-	(version 20250114)
+	(version 20260306)
 	(generator "eeschema")
-	(generator_version "9.0")
+	(generator_version "10.0")
 	(paper "A3")

Commit message: Update
Parts:
- R16, R17: value 10KΩ -> 2.2KΩ
- R22, R23: value 2.2KΩ -> 10KΩ
